Commit message: Added gazebo

File: install/pickplace_rl_mobile/share/pickplace_rl_mobile/urdf/pickplace_mobile_arm.urdf (robot description, URDF)
Before this commit: robot pickplace_rl_mobile, 13 links, 12 joints
Links:
- link camera_optical_frame: mass 0.01 -> None; geometry 

Commit message: add pick and place script and state machine rl

File: install/pickplace_rl_mobile/share/pickplace_rl_mobile/urdf/pickplace_mobile_arm.urdf (robot description, URDF)
Before this commit: robot pickplace_rl_mobile, 13 links, 12 joints
Links:
- added link dummy_root
- link arm_base: geometry collision cylinder length=0.1 radius=0.06; visual cylinder length=0.1 radius=0.06
- link arm_link1: geometry collision box size=0.06 0.08 0.24; visual box size=0.06 0.08 0.24
- link arm_link2: geometry collision box size=0.24 0.06 0.06; visual box size=0.24 0.06 0.06
- link arm_link3: geometry collision box size=0.2 0.04 0.04; visual box size=0.2 0.04 0.04
- link base_link: geometry collision box size=0.45 0.35 0.08; visual box size=0.4 0.3 0.01
- link camera_link: geometry collision box size=0.04 0.1 0.04; visual box size=0.04 0.1 0.04
- link ee_link: geometry collision box size=0.04 0.08 0.03; visual box size=0.04 0.08 0.03
- link left_finger: geometry collision box size=0.04 0.015 0.06; visual box size=0.03 0.002 0.05
- link left_wheel: geometry collision cylinder length=0.05 radius=0.08; visual cylinder length=0.005 radius=0.06
- link right_finger: geometry collision box size=0.04 0.015 0.06; visual box size=0.03 0.002 0.05
- link right_wheel: geometry collision cylinder length=0.05 radius=0.08; visual cylinder length=0.005 radius=0.06
- link wrist_link: geometry collision cylinder length=0.05 radius=0.025; visual cylinder length=0.05 radius=0.025
Joints:
- added joint dummy_joint: type fixed, parent dummy_root, child base_link
- joint arm_base_joint: origin xyz=0.1 0 0.1 rpy=0 0 0 -> xyz=-0.1 0 0.1 rpy=0 0 0
- joint camera_joint: origin xyz=0.15 0 0.15 rpy=0 0.2 0 -> xyz=0.22 0 0.05 rpy=0 0.3 0
- joint elbow_joint: origin xyz=0.2 0 0 rpy=0 0 0 -> xyz=0.24 0 0 rpy=0 0 0
- joint left_finger_joint: limit lower=0 upper=0.03 effort=5 velocity=0.1 -> lower=-0.01 upper=0.03 effort=5 velocity=0.1; origin xyz=0.03 0.02 0 rpy=0 0 0 -> xyz=0.02 0.03 0 rpy=0 0 0
- joint left_wheel_joint: origin xyz=0 0.165 0 rpy=0 0 0 -> xyz=0.1 0.205 0 rpy=0 0 0
- joint right_finger_joint: limit lower=0 upper=0.03 effort=5 velocity=0.1 -> lower=-0.01 upper=0.03 effort=5 velocity=0.1; origin xyz=0.03 -0.02 0 rpy=0 0 0 -> xyz=0.02 -0.03 0 rpy=0 0 0
- joint right_wheel_joint: origin xyz=0 -0.165 0 rpy=0 0 0 -> xyz=0.1 -0.205 0 rpy=0 0 0
- joint shoulder_pitch_joint: origin xyz=0 0 0.2 rpy=0 0 0 -> xyz=0 0 0.24 rpy=0 0 0
- joint wrist_pitch_joint: origin xyz=0 0 0.02 rpy=0 0 0 -> xyz=0.03 0 0 rpy=0 0 0
- joint wrist_roll_joint: origin xyz=0.16 0 0 rpy=0 0 0 -> xyz=0.2 0 0 rpy=0 0 0
