Commit message: Update URDF for mobile arm

File: src/pickplace_rl_mobile/urdf/pickplace_mobile_arm.urdf (robot description, URDF)
Before this commit: robot pickplace_rl_mobile, 14 links, 13 joints
Links:
- added link lidar_link, mass 0.05; collision cylinder length=0.04 radius=0.03; visual cylinder length=0.04 radius=0.03
Joints:
- added joint lidar_joint: type fixed, parent base_link, child lidar_link, origin xyz=0.0 0 0.12 rpy=0 0 0
